Commit message: More fixes and added gripper inertial properties

File: angler_description/urdf/alpha.ros2_control.xacro (robot description, xacro)
@@ -36,8 +36,5 @@
           <param name="initial_value">${initial_positions['axis_a']}</param>
         </state_interface>
-        <state_interface
-          name="velocity">
-          <param name="initial_value">0.0</param>
-        </state_interface>
+        <state_interface name="velocity" />
       </joint>
       <joint name="alpha_axis_b">
@@ -53,4 +50,5 @@
           <param name="initial_value">${initial_positions['axis_b']}</param>
         </state_interface>
+        <state_interface name="velocity" />
       </joint>
       <joint name="alpha_axis_c">
@@ -66,4 +64,5 @@
           <param name="initial_value">${initial_positions['axis_c']}</param>
         </state_interface>
+        <state_interface name="velocity" />
       </joint>
       <joint name="alpha_axis_d">
@@ -79,4 +78,5 @@
           <param name="initial_value">${initial_positions['axis_d']}</param>
         </state_interface>
+        <state_interface name="velocity" />
       </joint>
       <joint name="alpha_axis_e">
@@ -92,4 +92,5 @@
           <param name="initial_value">${initial_positions['axis_e']}</param>
         </state_interface>
+        <state_interface name="velocity" />
       </joint>
     </ros2_control>

File: angler_description/urdf/alpha.urdf.xacro (robot description, xacro)
@@ -32,4 +32,10 @@
         <material name="${prefix}black" />
       </visual>
+      <collision>
+        <geometry>
+          <cylinder length="0.150" radius="0.020" />
+        </geometry>
+        <origin rpy="0 1.57075 0" xyz="-0.055 0 0" />
+      </collision>
       <inertial>
         <mass value="0.341" />
@@ -53,4 +59,10 @@
         <material name="${prefix}black" />
       </visual>
+      <collision>
+        <geometry>
+          <cylinder length="0.033" radius="0.020" />
+        </geometry>
+        <origin rpy="0 0 0" xyz="0 0 0.0165" />
+      </collision>
       <inertial>
         <mass value="0.194" />
@@ -74,4 +86,22 @@
         <material name="${prefix}black" />
       </visual>
+      <collision>
+        <geometry>
+          <cylinder length="0.145" radius="0.020" />
+        </geometry>
+        <origin rpy="0 0 0" xyz="-0.02 0 -0.0725" />
+      </collision>
+      <collision>
+        <geometry>
+          <cylinder length="0.040" radius="0.020" />
+        </geometry>
+        <origin rpy="1.5707 0 0" xyz="0 0 0" />
+      </collision>
+      <collision>
+        <geometry>
+          <cylinder length="0.040" radius="0.020" />
+        </geometry>
+        <origin rpy="1.5707 0 0" xyz="-0.040 0 -0.1453" />
+      </collision>
       <inertial>
         <mass value="0.429" />
@@ -95,4 +125,10 @@
         <material name="${prefix}black" />
       </visual>
+      <collision>
+        <geometry>
+          <cylinder length="0.033" radius="0.020" />
+        </geometry>
+        <origin rpy="0 0 0" xyz="0.02 0 0.0165" />
+      </collision>
       <inertial>
         <mass value="0.115" />
@@ -117,14 +153,20 @@
         <material name="${prefix}black" />
       </visual>
-      <inertial>
-        <mass value="0.333" />
-        <origin xyz="0 0 0.054875" />
-        <inertia
-          ixx="0.0003676"
-          ixy="0"
-          ixz="0"
-          iyy="0.0003676"
-          iyz="0"
-          izz="0.0000666"
+      <collision>
+        <geometry>
+          <cylinder length="0.1" radius="0.020" />
+        </geometry>
+        <origin rpy="0 0 0" xyz="0 0 0.05" />
+      </collision>
+      <inertial>
+        <mass value="0.200" />
+        <origin xyz="0 0 0.05" />
+        <inertia
+          ixx="0.0001867"
+          ixy="0"
+          ixz="0"
+          iyy="0.0001867"
+          iyz="0"
+          izz="0.00004"
         />
       </inertial>

File: angler_description/urdf/angler.config.xacro (robot description, xacro)
@@ -9,4 +9,5 @@
   <xacro:arg name="initial_positions_file" default="initial_positions.yaml" />
   <xacro:arg name="namespace" default="" />
+  <xacro:arg name="use_sim" default="false" />
   <!-- Import BlueROV2 Heavy macro -->
   <xacro:include filename="$(find angler_description)/urdf/bluerov2_heavy_modified.urdf.xacro" />
@@ -19,5 +20,5 @@
     name="ReachAlpha5" use_fake_hardware="$(arg use_fake_hardware)" serial_port="$(arg serial_port)"
     state_update_frequency="$(arg state_update_frequency)"
-    initial_positions_file="$(arg initial_positions_file)" />
+    initial_positions_file="$(arg initial_positions_file)" use_sim="$(arg use_sim)" />
   <xacro:if value="$(arg use_sim)">
     <xacro:angler_gazebo prefix="$(arg prefix)" namespace="$(arg namespace)"

File: angler_description/urdf/end_effectors/standard_jaws.urdf.xacro (robot description, xacro)
@@ -14,13 +14,20 @@
         <material name="${prefix}black" />
       </visual>
+      <collision>
+        <geometry>
+          <cylinder length="0.00975" radius="0.020" />
+        </geometry>
+        <origin rpy="0 0 0" xyz="0 0 0.004875" />
+      </collision>
       <inertial>
-        <mass value="0.0001" />
+        <mass value="0.023" />
+        <origin xyz="0 0 0.004875" />
         <inertia
-          ixx="0.0001"
+          ixx="0.000002422"
           ixy="0"
           ixz="0"
-          iyy="0.0001"
+          iyy="0.000002422"
           iyz="0"
-          izz="0.0001"
+          izz="0.0000046"
         />
       </inertial>
@@ -35,13 +42,20 @@
         <origin xyz="0 0 0" rpy="0 0 0" />
       </visual>
+      <collision>
+        <geometry>
+          <box size="0.012 0.03 0.09" />
+        </geometry>
+        <origin xyz="0.0 -0.008 0.045" rpy="0 0 0" />
+      </collision>
       <inertial>
-        <mass value="0.0001" />
+        <mass value="0.055" />
+        <origin xyz="0.0 -0.008 0.045" rpy="0 0 0" />
         <inertia
-          ixx="0.0001"
+          ixx="0.00004125"
           ixy="0"
           ixz="0"
-          iyy="0.0001"
+          iyy="0.000037785"
           iyz="0"
-          izz="0.0001"
+          izz="0.000004785"
         />
       </inertial>
@@ -56,13 +70,20 @@
         <origin xyz="0 0 0" rpy="0 0 0" />
       </visual>
+      <collision>
+        <geometry>
+          <box size="0.012 0.03 0.09" />
+        </geometry>
+        <origin xyz="0.0 0.008 0.045" rpy="0 0 0" />
+      </collision>
       <inertial>
-        <mass value="0.0001" />
+        <mass value="0.055" />
+        <origin xyz="0.0 0.008 0.045" rpy="0 0 0" />
         <inertia
-          ixx="0.0001"
+          ixx="0.00004125"
           ixy="0"
           ixz="0"
-          iyy="0.0001"
+          iyy="0.000037785"
           iyz="0"
-          izz="0.0001"
+          izz="0.000004785"
         />
       </inertial>
