Commit message: Fixed axis d bug, resolved solution selection bug, and added nvidia driver support

File: angler_description/urdf/alpha.urdf.xacro (robot description, xacro)
@@ -233,5 +233,6 @@
       <origin xyz="-0.02 0 0.033" />
       <axis xyz="0 1 0" />
-      <limit effort="9.0" lower="0.0" upper="3.49" velocity="0.5" />
+      <!-- The true lower limit is 0.0; however, this breaks for some reason with ros2_control -->
+      <limit effort="9.0" lower="-3.49" upper="3.49" velocity="0.5" />
     </joint>
     <joint name="${prefix}axis_c" type="revolute">
