Commit message: fixed bouyancy for bluerov2

File: angler_description/urdf/bluerov2_heavy_modified.urdf.xacro (robot description, xacro)
@@ -25,9 +25,33 @@
         <origin rpy="0 0 0" xyz="0 0 0" />
       </visual>
+      <!-- Split the collision into four boxes so that
+      we can adjust each one to balance things out -->
+      <!-- Front left -->
       <collision>
         <geometry>
-          <box size="0.457 0.575 0.05" />
-        </geometry>
-        <origin rpy="0 0 0" xyz="0 0 0.06" />
+          <box size="0.2285 0.2875 0.071" />
+        </geometry>
+        <origin rpy="0 0 0" xyz="0.11425 0.14375 0.08" />
+      </collision>
+      <!-- Front right -->
+      <collision>
+        <geometry>
+          <box size="0.2285 0.2875 0.081" />
+        </geometry>
+        <origin rpy="0 0 0" xyz="0.11425 -0.14375 0.08" />
+      </collision>
+      <!-- Back left -->
+      <collision>
+        <geometry>
+          <box size="0.2285 0.2875 0.051" />
+        </geometry>
+        <origin rpy="0 0 0" xyz="-0.11425 0.14375 0.08" />
+      </collision>
+      <!-- Back right -->
+      <collision>
+        <geometry>
+          <box size="0.2285 0.2875 0.061" />
+        </geometry>
+        <origin rpy="0 0 0" xyz="-0.11425 -0.14375 0.08" />
       </collision>
     </link>

Commit message: WHY WONT THE POSITION JACOBIAN WORK FOR THE LOVE OF GOD

File: angler_description/urdf/bluerov2_heavy_modified.urdf.xacro (robot description, xacro)
@@ -30,5 +30,5 @@
       <collision>
         <geometry>
-          <box size="0.2285 0.2875 0.071" />
+          <box size="0.2285 0.2875 0.075" />
         </geometry>
         <origin rpy="0 0 0" xyz="0.11425 0.14375 0.08" />
@@ -37,5 +37,5 @@
       <collision>
         <geometry>
-          <box size="0.2285 0.2875 0.081" />
+          <box size="0.2285 0.2875 0.085" />
         </geometry>
         <origin rpy="0 0 0" xyz="0.11425 -0.14375 0.08" />

File: angler_description/urdf/end_effectors/standard_jaws.urdf.xacro (robot description, xacro)
@@ -89,4 +89,23 @@
       </inertial>
     </link>
+    <link name="${prefix}tool">
+      <visual>
+        <origin rpy="0 0 0" xyz="0 0 0" />
+        <geometry>
+          <box size="0.001 0.001 0.001" />
+        </geometry>
+      </visual>
+      <inertial>
+        <mass value="0.0001" />
+        <inertia
+          ixx="0.0001"
+          ixy="0"
+          ixz="0"
+          iyy="0.0001"
+          iyz="0"
+          izz="0.0001"
+        />
+      </inertial>
+    </link>
     <joint name="${prefix}base_joint" type="fixed">
       <xacro:insert_block name="origin" />
@@ -111,4 +130,9 @@
       <mimic joint="${prefix}rs1_130_joint" multiplier="1" offset="0" />
     </joint>
+    <joint name="${prefix}tool_joint" type="fixed">
+      <origin xyz="0 0 0.04" rpy="0 -1.571 0" />
+      <parent link="${prefix}base_link" />
+      <child link="${prefix}tool" />
+    </joint>
   </xacro:macro>
 </robot>
