Commit message: Continued integrating uvms model

File: angler_description/config/angler.config.xacro (robot description, xacro)
@@ -11,10 +11,10 @@
   <xacro:arg name="namespace" default="" />
   <!-- Import BlueROV2 Heavy macro -->
-  <xacro:include filename="$(find angler_description)/urdf/bluerov2_heavy.urdf.xacro" />
+  <xacro:include filename="$(find angler_description)/urdf/bluerov2_heavy_modified.urdf.xacro" />
   <!-- Import ros2_control macro -->
   <xacro:include filename="$(find angler_description)/ros2_control/alpha.ros2_control.xacro" />
   <!-- Import Gazebo macro -->
   <xacro:include filename="$(find angler_description)/gazebo/angler.gazebo.xacro" />
-  <xacro:bluerov2_heavy_urdf prefix="$(arg prefix)" />
+  <xacro:bluerov2_heavy_modified_urdf prefix="$(arg prefix)" />
   <xacro:if value="$(arg use_sim)">
     <xacro:angler_gazebo prefix="$(arg prefix)" controllers_file="$(arg controllers_file)"

File: angler_description/gazebo/angler.gazebo.xacro (robot description, xacro)
@@ -11,14 +11,4 @@
         <update_rate>1000.0</update_rate>
         <topic>__default_topic__</topic>
-        <plugin filename="libgazebo_ros_imu_sensor.so" name="imu_plugin">
-          <topicName>imu</topicName>
-          <bodyName>imu_link</bodyName>
-          <updateRateHZ>1000.0</updateRateHZ>
-          <gaussianNoise>0.0</gaussianNoise>
-          <xyzOffset>0 0 0</xyzOffset>
-          <rpyOffset>0 0 0</rpyOffset>
-          <frameName>imu_link</frameName>
-          <initialOrientationAsReference>false</initialOrientationAsReference>
-        </plugin>
       </sensor>
     </gazebo>
@@ -279,36 +269,36 @@
       </plugin>
     </gazebo>
-    <gazebo reference="${prefix}alpha/base_link">
-      <material>Gazebo/Gray</material>
-    </gazebo>
-    <gazebo reference="${prefix}alpha/ee_base_link">
-      <material>Gazebo/Gray</material>
-    </gazebo>
-    <gazebo reference="${prefix}alpha/m1_link" />
-    <gazebo reference="${prefix}alpha/m1_link">
-      <material>Gazebo/Gray</material>
-    </gazebo>
-    <gazebo reference="${prefix}alpha/m2_1_1_link">
-      <material>Gazebo/Gray</material>
-    </gazebo>
-    <gazebo reference="${prefix}alpha/m2_1_2_link">
-      <material>Gazebo/Gray</material>
-    </gazebo>
-    <gazebo reference="${prefix}alpha/m2_joint_link">
-      <material>Gazebo/Gray</material>
-    </gazebo>
-    <gazebo reference="${prefix}alpha/m3_inline_link">
-      <material>Gazebo/Gray</material>
-    </gazebo>
-    <gazebo reference="${prefix}alpha/push_rod">
-      <material>Gazebo/Gray</material>
-    </gazebo>
-    <gazebo reference="${prefix}alpha/standard_jaws_base_link">
-      <material>Gazebo/Gray</material>
-    </gazebo>
-    <gazebo reference="${prefix}alpha/standard_jaws_rs1_130_link">
-      <material>Gazebo/Gray</material>
-    </gazebo>
-    <gazebo reference="${prefix}alpha/standard_jaws_rs1_139_link">
+    <gazebo reference="${prefix}alpha_base_link">
+      <material>Gazebo/Gray</material>
+    </gazebo>
+    <gazebo reference="${prefix}alpha_ee_base_link">
+      <material>Gazebo/Gray</material>
+    </gazebo>
+    <gazebo reference="${prefix}alpha_m1_link" />
+    <gazebo reference="${prefix}alpha_m1_link">
+      <material>Gazebo/Gray</material>
+    </gazebo>
+    <gazebo reference="${prefix}alpha_m2_1_1_link">
+      <material>Gazebo/Gray</material>
+    </gazebo>
+    <gazebo reference="${prefix}alpha_m2_1_2_link">
+      <material>Gazebo/Gray</material>
+    </gazebo>
+    <gazebo reference="${prefix}alpha_m2_joint_link">
+      <material>Gazebo/Gray</material>
+    </gazebo>
+    <gazebo reference="${prefix}alpha_m3_inline_link">
+      <material>Gazebo/Gray</material>
+    </gazebo>
+    <gazebo reference="${prefix}alpha_push_rod">
+      <material>Gazebo/Gray</material>
+    </gazebo>
+    <gazebo reference="${prefix}alpha_standard_jaws_base_link">
+      <material>Gazebo/Gray</material>
+    </gazebo>
+    <gazebo reference="${prefix}alpha_standard_jaws_rs1_130_link">
+      <material>Gazebo/Gray</material>
+    </gazebo>
+    <gazebo reference="${prefix}alpha_standard_jaws_rs1_139_link">
       <material>Gazebo/Gray</material>
     </gazebo>

Commit message: Started to cleanup dockerfile to fix gz launch bugs

File: angler_description/config/angler.config.xacro (robot description, xacro)
@@ -7,5 +7,5 @@
   <xacro:arg name="serial_port" default="" />
   <xacro:arg name="state_update_frequency" default="250" />
-  <xacro:arg name="controllers_file" default="alpha_controllers.yaml" />
+  <xacro:arg name="controllers_file" default="angler_controllers.yaml" />
   <xacro:arg name="initial_positions_file" default="initial_positions.yaml" />
   <xacro:arg name="namespace" default="" />
@@ -18,6 +18,6 @@
   <xacro:bluerov2_heavy_modified_urdf prefix="$(arg prefix)" />
   <xacro:if value="$(arg use_sim)">
-    <xacro:angler_gazebo prefix="$(arg prefix)" controllers_file="$(arg controllers_file)"
-      namespace="$(arg namespace)" />
+    <xacro:angler_gazebo prefix="$(arg prefix)" namespace="$(arg namespace)"
+      controllers_file="$(arg controllers_file)" />
   </xacro:if>
   <xacro:alpha_system

File: angler_description/gazebo/angler.gazebo.xacro (robot description, xacro)
@@ -1,306 +1,18 @@
 <?xml version="1.0"?>
 <robot xmlns:xacro="http://ros.org/wiki/xacro">
-  <xacro:macro name="angler_gazebo" params="prefix namespace">
-    <!-- IMU sensor gyro and accel data will be sent to ArduSub -->
-    <gazebo reference="${prefix}base_link">
-      <sensor name="imu_sensor" type="imu">
-        <!-- Transform from the Gazebo body frame (x-forward, y-left, z-up)
-             to the ArduPilot body frame (x-forward, y-right, z-down) -->
-        <pose>0 0 0 3.142 0 0</pose>
-        <always_on>true</always_on>
-        <update_rate>1000.0</update_rate>
-        <topic>__default_topic__</topic>
-      </sensor>
-    </gazebo>
-    <!-- Hydrodynamics plugin -->
-    <gazebo>
-      <plugin
-        filename="gz-sim-hydrodynamics-system"
-        name="gz::sim::systems::Hydrodynamics">
-        <link_name>${prefix}base_link</link_name>
-        <water_density>1000.0</water_density>
-        <!-- Added mass: -->
-        <xDotU>0</xDotU>
-        <yDotV>0</yDotV>
-        <zDotW>0</zDotW>
-        <kDotP>0</kDotP>
-        <mDotQ>0</mDotQ>
-        <nDotR>0</nDotR>
-        <!-- First order stability derivative: -->
-        <xU>0</xU>
-        <yV>0</yV>
-        <zW>0</zW>
-        <kP>0</kP>
-        <mQ>0</mQ>
-        <nR>0</nR>
-        <!-- Second order stability derivative: -->
-        <xUabsU>-58.42</xUabsU>
-        <yVabsV>-55.137</yVabsV>
-        <zWabsW>-124.818</zWabsW>
-        <kPabsP>-4.0</kPabsP>
-        <mQabsQ>-4.0</mQabsQ>
-        <nRabsR>-4.0</nRabsR>
-      </plugin>
-    </gazebo>
-    <!-- Thruster plugins -->
-    <gazebo>
-      <plugin
-        filename="gz-sim-thruster-system"
-        name="gz::sim::systems::Thruster">
-        <namespace>${namespace}</namespace>
-        <joint_name>${prefix}thruster1_joint</joint_name>
-        <thrust_coefficient>0.02</thrust_coefficient>
-        <fluid_density>1000.0</fluid_density>
-        <propeller_diameter>0.1</propeller_diameter>
-        <velocity_control>true</velocity_control>
-        <use_angvel_cmd>False</use_angvel_cmd>
-      </plugin>
-    </gazebo>
-    <gazebo>
-      <plugin
-        filename="gz-sim-thruster-system"
-        name="gz::sim::systems::Thruster">
-        <namespace>${namespace}</namespace>
-        <joint_name>${prefix}thruster2_joint</joint_name>
-        <thrust_coefficient>0.02</thrust_coefficient>
-        <fluid_density>1000.0</fluid_density>
-        <propeller_diameter>0.1</propeller_diameter>
-        <velocity_control>true</velocity_control>
-        <use_angvel_cmd>False</use_angvel_cmd>
-      </plugin>
-    </gazebo>
-    <gazebo>
-      <plugin
-        filename="gz-sim-thruster-system"
-        name="gz::sim::systems::Thruster">
-        <namespace>${namespace}</namespace>
-        <joint_name>${prefix}thruster3_joint</joint_name>
-        <!-- Reverse spin to balance torque -->
-        <thrust_coefficient>-0.02</thrust_coefficient>
-        <fluid_density>1000.0</fluid_density>
-        <propeller_diameter>0.1</propeller_diameter>
-        <velocity_control>true</velocity_control>
-        <use_angvel_cmd>False</use_angvel_cmd>
-      </plugin>
-    </gazebo>
-    <gazebo>
-      <plugin
-        filename="gz-sim-thruster-system"
-        name="gz::sim::systems::Thruster">
-        <namespace>${namespace}</namespace>
-        <joint_name>${prefix}thruster4_joint</joint_name>
-        <!-- Reverse spin to balance torque -->
-        <thrust_coefficient>-0.02</thrust_coefficient>
-        <fluid_density>1000.0</fluid_density>
-        <propeller_diameter>0.1</propeller_diameter>
-        <velocity_control>true</velocity_control>
-        <use_angvel_cmd>False</use_angvel_cmd>
-      </plugin>
-    </gazebo>
-    <gazebo>
-      <plugin
-        filename="gz-sim-thruster-system"
-        name="gz::sim::systems::Thruster">
-        <namespace>${namespace}</namespace>
-        <joint_name>${prefix}thruster5_joint</joint_name>
-        <thrust_coefficient>0.02</thrust_coefficient>
-        <fluid_density>1000.0</fluid_density>
-        <propeller_diameter>0.1</propeller_diameter>
-        <velocity_control>true</velocity_control>
-        <use_angvel_cmd>False</use_angvel_cmd>
-      </plugin>
-    </gazebo>
-    <gazebo>
-      <plugin
-        filename="gz-sim-thruster-system"
-        name="gz::sim::systems::Thruster">
-        <namespace>${namespace}</namespace>
-        <joint_name>${prefix}thruster6_joint</joint_name>
-        <!-- Reverse spin to balance torque -->
-        <thrust_coefficient>-0.02</thrust_coefficient>
-        <fluid_density>1000.0</fluid_density>
-        <propeller_diameter>0.1</propeller_diameter>
-        <velocity_control>true</velocity_control>
-        <use_angvel_cmd>False</use_angvel_cmd>
-      </plugin>
-    </gazebo>
-    <gazebo>
-      <plugin
-        filename="gz-sim-thruster-system"
-        name="gz::sim::systems::Thruster">
-        <namespace>${namespace}</namespace>
-        <joint_name>${prefix}thruster7_joint</joint_name>
-        <!-- Reverse spin to balance torque -->
-        <thrust_coefficient>-0.02</thrust_coefficient>
-        <fluid_density>1000.0</fluid_density>
-        <propeller_diameter>0.1</propeller_diameter>
-        <velocity_control>true</velocity_control>
-        <use_angvel_cmd>False</use_angvel_cmd>
-      </plugin>
-    </gazebo>
-    <gazebo>
-      <plugin
-        filename="gz-sim-thruster-system"
-        name="gz::sim::systems::Thruster">
-        <namespace>${namespace}</namespace>
-        <joint_name>${prefix}thruster8_joint</joint_name>
-        <thrust_coefficient>0.02</thrust_coefficient>
-        <fluid_density>1000.0</fluid_density>
-        <propeller_diameter>0.1</propeller_diameter>
-        <velocity_control>true</velocity_control>
-        <use_angvel_cmd>False</use_angvel_cmd>
-      </plugin>
-    </gazebo>
-    <!-- Ardupilot -->
-    <gazebo>
-      <plugin name="ArduPilotPlugin" filename="libArduPilotPlugin.so">
-        <!-- Port settings -->
-        <fdm_addr>127.0.0.1</fdm_addr>
-        <fdm_port_in>9002</fdm_port_in>
-        <connectionTimeoutMaxCount>5</connectionTimeoutMaxCount>
-        <lock_step>1</lock_step>
-        <!-- Transform from the Gazebo body frame (x-forward, y-left, z-up)
-           to the ArduPilot body frame (x-forward, y-right, z-down) -->
-        <modelXYZToAirplaneXForwardZDown>0 0 0 3.142 0 0</modelXYZToAirplaneXForwardZDown>
-        <!-- Transform from the Gazebo world frame (ENU)
-           to the ArduPilot world frame (NED) -->
-        <gazeboXYZToNED>0 0 0 3.142 0 1.571</gazeboXYZToNED>
-        <!-- Sensors -->
-        <imuName>imu_sensor</imuName>
-        <!-- Thrusters -->
-        <control channel="0">
-          <jointName>${prefix}thruster1_joint</jointName>
-          <servo_min>1100</servo_min>
-          <servo_max>1900</servo_max>
-          <type>COMMAND</type>
-          <cmd_topic>/model/${namespace}/joint/${prefix}thruster1_joint/cmd_thrust</cmd_topic>
-          <offset>-0.5</offset>
-          <multiplier>100</multiplier>
-        </control>
-        <control channel="1">
-          <jointName>${prefix}thruster2_joint</jointName>
-          <servo_min>1100</servo_min>
-          <servo_max>1900</servo_max>
-          <type>COMMAND</type>
-          <cmd_topic>/model/${namespace}/joint/${prefix}thruster2_joint/cmd_thrust</cmd_topic>
-          <offset>-0.5</offset>
-          <multiplier>100</multiplier>
-        </control>
-        <control channel="2">
-          <jointName>${prefix}thruster3_joint</jointName>
-          <servo_min>1100</servo_min>
-          <servo_max>1900</servo_max>
-          <type>COMMAND</type>
-          <cmd_topic>/model/${namespace}/joint/${prefix}thruster3_joint/cmd_thrust</cmd_topic>
-          <offset>-0.5</offset>
-          <multiplier>100</multiplier>
-        </control>
-        <control channel="3">
-          <jointName>${prefix}thruster4_joint</jointName>
-          <servo_min>1100</servo_min>
-          <servo_max>1900</servo_max>
-          <type>COMMAND</type>
-          <cmd_topic>/model/${namespace}/joint/${prefix}thruster4_joint/cmd_thrust</cmd_topic>
-          <offset>-0.5</offset>
-          <multiplier>100</multiplier>
-        </control>
-        <control channel="4">
-          <jointName>${prefix}thruster5_joint</jointName>
-          <servo_min>1100</servo_min>
-          <servo_max>1900</servo_max>
-          <type>COMMAND</type>
-          <cmd_topic>/model/${namespace}/joint/${prefix}thruster5_joint/cmd_thrust</cmd_topic>
-          <offset>-0.5</offset>
-          <multiplier>100</multiplier>
-        </control>
-        <control channel="5">
-          <jointName>${prefix}thruster6_joint</jointName>
-          <servo_min>1100</servo_min>
-          <servo_max>1900</servo_max>
-          <type>COMMAND</type>
-          <cmd_topic>/model/${namespace}/joint/${prefix}thruster6_joint/cmd_thrust</cmd_topic>
-          <offset>-0.5</offset>
-          <multiplier>100</multiplier>
-        </control>
-        <control channel="6">
-          <jointName>${prefix}thruster7_joint</jointName>
-          <servo_min>1100</servo_min>
-          <servo_max>1900</servo_max>
-          <type>COMMAND</type>
-          <cmd_topic>/model/${namespace}/joint/${prefix}thruster7_joint/cmd_thrust</cmd_topic>
-          <offset>-0.5</offset>
-          <multiplier>100</multiplier>
-        </control>
-        <control channel="7">
-          <jointName>${prefix}thruster8_joint</jointName>
-          <servo_min>1100</servo_min>
-          <servo_max>1900</servo_max>
-          <type>COMMAND</type>
-          <cmd_topic>/model/${namespace}/joint/${prefix}thruster8_joint/cmd_thrust</cmd_topic>
-          <offset>-0.5</offset>
-          <multiplier>100</multiplier>
-        </control>
-      </plugin>
-    </gazebo>
-    <!-- Publish the ground-truth pose -->
-    <gazebo>
-      <plugin
-        filename="gz-sim-odometry-publisher-system"
-        name="gz::sim::systems::OdometryPublisher">
-        <odom_frame>map</odom_frame>
-        <robot_base_frame>${prefix}base_link</robot_base_frame>
-        <dimensions>3</dimensions>
-        <odom_publish_frequency>100</odom_publish_frequency>
-      </plugin>
-    </gazebo>
-    <!-- Setup ros2_control for the Alpha -->
-    <gazebo>
-      <plugin
-        filename="libgz_ros2_control-system.so"
-        name="gz_ros2_control::GazeboSimROS2ControlPlugin">
-        <xacro:if value="${namespace != '/'}">
-          <ros>
-            <namespace>/${namespace[:-1]}</namespace>
-          </ros>
-          <robot_param_node>/${namespace}robot_state_publisher</robot_param_node>
-        </xacro:if>
-        <parameters>
-          $(find angler_description)/config/${controllers_file}</parameters>
-      </plugin>
-    </gazebo>
-    <gazebo reference="${prefix}alpha_base_link">
-      <material>Gazebo/Gray</material>
-    </gazebo>
-    <gazebo reference="${prefix}alpha_ee_base_link">
-      <material>Gazebo/Gray</material>
-    </gazebo>
-    <gazebo reference="${prefix}alpha_m1_link" />
-    <gazebo reference="${prefix}alpha_m1_link">
-      <material>Gazebo/Gray</material>
-    </gazebo>
-    <gazebo reference="${prefix}alpha_m2_1_1_link">
-      <material>Gazebo/Gray</material>
-    </gazebo>
-    <gazebo reference="${prefix}alpha_m2_1_2_link">
-      <material>Gazebo/Gray</material>
-    </gazebo>
-    <gazebo reference="${prefix}alpha_m2_joint_link">
-      <material>Gazebo/Gray</material>
-    </gazebo>
-    <gazebo reference="${prefix}alpha_m3_inline_link">
-      <material>Gazebo/Gray</material>
-    </gazebo>
-    <gazebo reference="${prefix}alpha_push_rod">
-      <material>Gazebo/Gray</material>
-    </gazebo>
-    <gazebo reference="${prefix}alpha_standard_jaws_base_link">
-      <material>Gazebo/Gray</material>
-    </gazebo>
-    <gazebo reference="${prefix}alpha_standard_jaws_rs1_130_link">
-      <material>Gazebo/Gray</material>
-    </gazebo>
-    <gazebo reference="${prefix}alpha_standard_jaws_rs1_139_link">
-      <material>Gazebo/Gray</material>
-    </gazebo>
+  <xacro:macro name="angler_gazebo" params="prefix namespace controllers_file">
+    <xacro:include filename="$(find angler_description)/gazebo/ardupilot.gazebo.xacro" />
+    <xacro:include filename="$(find angler_description)/gazebo/hydrodynamics.gazebo.xacro" />
+    <xacro:include filename="$(find angler_description)/gazebo/materials.gazebo.xacro" />
+    <xacro:include filename="$(find angler_description)/gazebo/ros2_control.gazebo.xacro" />
+    <xacro:include filename="$(find angler_description)/gazebo/sensors.gazebo.xacro" />
+    <xacro:include filename="$(find angler_description)/gazebo/thrusters.gazebo.xacro" />
+    <xacro:ardupilot prefix="$(arg prefix)" namespace="$(arg namespace)" />
+    <xacro:hydrodynamics prefix="$(arg prefix)" />
+    <xacro:materials prefix="$(arg prefix)" />
+    <xacro:ros2_control namespace="$(arg namespace)" controllers_file="$(arg controllers_file)" />
+    <xacro:imu prefix="$(arg prefix)" />
+    <xacro:odom prefix="$(arg prefix)" />
+    <xacro:thrusters prefix="$(arg prefix)" namespace="$(arg namespace)" />
   </xacro:macro>
 </robot>

File: angler_description/ros2_control/alpha.ros2_control.xacro (robot description, xacro)
@@ -8,5 +8,5 @@
       <xacro:if value="$(arg use_sim)">
         <hardware>
-          <plugin>gazebo_ros2_control/GazeboSystem</plugin>
+          <plugin>gz_ros2_control/GazeboSimSystem</plugin>
         </hardware>
       </xacro:if>
