Commit message: [wip] resolved ros2_control launch issues - currently breaking down into smaller files

File: angler_description/config/angler.config.xacro (robot description, xacro)
@@ -4,5 +4,4 @@
   <xacro:arg name="prefix" default="" />
   <xacro:arg name="use_fake_hardware" default="true" />
-  <xacro:arg name="use_sim" default="false" />
   <xacro:arg name="serial_port" default="" />
   <xacro:arg name="state_update_frequency" default="250" />
@@ -13,15 +12,13 @@
   <xacro:include filename="$(find angler_description)/urdf/bluerov2_heavy_modified.urdf.xacro" />
   <!-- Import ros2_control macro -->
-  <xacro:include filename="$(find angler_description)/ros2_control/alpha.ros2_control.xacro" />
+  <xacro:include filename="$(find angler_description)/urdf/alpha.ros2_control.xacro" />
   <!-- Import Gazebo macro -->
-  <xacro:include filename="$(find angler_description)/gazebo/angler.gazebo.xacro" />
+  <xacro:include filename="$(find angler_description)/urdf/angler.gazebo.xacro" />
   <xacro:bluerov2_heavy_modified_urdf prefix="$(arg prefix)" />
-  <xacro:if value="$(arg use_sim)">
-    <xacro:angler_gazebo prefix="$(arg prefix)" namespace="$(arg namespace)"
-      controllers_file="$(arg controllers_file)" />
-  </xacro:if>
   <xacro:alpha_system
     name="ReachAlpha5" use_fake_hardware="$(arg use_fake_hardware)" serial_port="$(arg serial_port)"
     state_update_frequency="$(arg state_update_frequency)"
-    initial_positions_file="$(arg initial_positions_file)" use_sim="$(arg use_sim)" />
+    initial_positions_file="$(arg initial_positions_file)" />
+  <xacro:angler_gazebo prefix="$(arg prefix)" namespace="$(arg namespace)"
+    controllers_file="$(arg controllers_file)" />
 </robot>

File: angler_description/urdf/alpha.ros2_control.xacro (robot description, xacro)
@@ -2,26 +2,11 @@
 <robot xmlns:xacro="http://www.ros.org/wiki/xacro">
   <xacro:macro name="alpha_system"
-    params="name serial_port state_update_frequency initial_positions_file use_sim:=^|false use_fake_hardware:=^true">
+    params="name serial_port state_update_frequency initial_positions_file use_fake_hardware:=^true">
     <xacro:property name="initial_positions"
-      value="${xacro.load_yaml(initial_positions_file)['initial_positions']}" />
+      value="${xacro.load_yaml('$(find angler_description)/config/$(arg initial_positions_file)')['initial_positions']}" />
     <ros2_control name="${name}" type="system">
-      <xacro:if value="$(arg use_sim)">
-        <hardware>
-          <plugin>gz_ros2_control/GazeboSimSystem</plugin>
-        </hardware>
-      </xacro:if>
-      <xacro:unless
-        value="$(arg use_sim)">
-        <hardware>
-          <xacro:if value="${use_fake_hardware}">
-            <plugin>mock_components/GenericSystem</plugin>
-          </xacro:if>
-          <xacro:unless value="${use_fake_hardware}">
-            <plugin>alpha_hardware/AlphaHardware</plugin>
-            <param name="serial_port">${serial_port}</param>
-            <param name="state_update_frequency">${state_update_frequency}</param>
-          </xacro:unless>
-        </hardware>
-      </xacro:unless>
+      <hardware>
+        <plugin>gz_ros2_control/GazeboSimSystem</plugin>
+      </hardware>
       <joint name="alpha_axis_a">
         <command_interface name="position">
@@ -34,5 +19,5 @@
         </command_interface>
         <state_interface name="position">
-          <param name="initial_value">${initial_positions['alpha_axis_a']}</param>
+          <param name="initial_value">${initial_positions['axis_a']}</param>
         </state_interface>
         <state_interface
@@ -51,8 +36,5 @@
         </command_interface>
         <state_interface name="position">
-          <param name="initial_value">${initial_positions['alpha_axis_b']}</param>
-        </state_interface>
-        <state_interface name="velocity">
-          <param name="initial_value">0.0</param>
+          <param name="initial_value">${initial_positions['axis_b']}</param>
         </state_interface>
       </joint>
@@ -67,8 +49,5 @@
         </command_interface>
         <state_interface name="position">
-          <param name="initial_value">${initial_positions['alpha_axis_c']}</param>
-        </state_interface>
-        <state_interface name="velocity">
-          <param name="initial_value">0.0</param>
+          <param name="initial_value">${initial_positions['axis_c']}</param>
         </state_interface>
       </joint>
@@ -83,8 +62,5 @@
         </command_interface>
         <state_interface name="position">
-          <param name="initial_value">${initial_positions['alpha_axis_d']}</param>
-        </state_interface>
-        <state_interface name="velocity">
-          <param name="initial_value">0.0</param>
+          <param name="initial_value">${initial_positions['axis_d']}</param>
         </state_interface>
       </joint>
@@ -99,8 +75,5 @@
         </command_interface>
         <state_interface name="position">
-          <param name="initial_value">${initial_positions['alpha_axis_e']}</param>
-        </state_interface>
-        <state_interface name="velocity">
-          <param name="initial_value">0.0</param>
+          <param name="initial_value">${initial_positions['axis_e']}</param>
         </state_interface>
       </joint>

File: angler_description/urdf/alpha.urdf.xacro (robot description, xacro)
@@ -5,28 +5,42 @@
       <color rgba="0.3 0.3 0.3 1" />
     </material>
-    <link name="${prefix}base_link" />
+    <link name="${prefix}base_link">
+      <visual>
+        <origin rpy="0 0 0" xyz="0 0 0" />
+        <geometry>
+          <box size="0.001 0.001 0.001" />
+        </geometry>
+      </visual>
+      <inertial>
+        <mass value="0.0001" />
+        <inertia
+          ixx="0.0001"
+          ixy="0"
+          ixz="0"
+          iyy="0.0001"
+          iyz="0"
+          izz="0.0001"
+        />
+      </inertial>
+    </link>
     <link name="${prefix}m3_inline_link">
       <visual>
         <geometry>
-          <mesh filename="package://alpha_description/meshes/M3-INLINE.stl" />
-        </geometry>
-        <origin rpy="0 0 0" xyz="0 0 0" />
-        <material name="${prefix}black" />
-      </visual>
-      <collision>
-        <geometry>
-          <cylinder length="0.150" radius="0.020" />
-        </geometry>
-      </collision>
+          <mesh filename="file://$(find alpha_description)/meshes/M3-INLINE.stl" />
+        </geometry>
+        <origin rpy="0 0 0" xyz="0 0 0" />
+        <material name="${prefix}black" />
+      </visual>
       <inertial>
         <mass value="0.341" />
-        <origin xyz="-0.075 -0.006 -0.003" />
-        <inertia
-          ixx="0.000099"
-          ixy="0.000139"
-          ixz="0.000115"
-          iyy="0.00292"
-          iyz="0.000003"
-          izz="0.002934" />
+        <origin xyz="-0.055 0 0" />
+        <inertia
+          ixx="0.0000682"
+          ixy="0"
+          ixz="0"
+          iyy="0.000673"
+          iyz="0"
+          izz="0.000673"
+        />
       </inertial>
     </link>
@@ -34,22 +48,20 @@
       <visual>
         <geometry>
-          <mesh filename="package://alpha_description/meshes/M2-1-1.stl" />
-        </geometry>
-        <origin rpy="0 0 0" xyz="0 0 0" />
-        <material name="${prefix}black" />
-      </visual>
-      <collision>
-        <geometry>
-          <cylinder length="0.066" radius="0.020" />
-        </geometry>
-        <origin rpy="0 0 0" xyz="0 0 0.000" />
-      </collision>
+          <mesh filename="file://$(find alpha_description)/meshes/M2-1-1.stl" />
+        </geometry>
+        <origin rpy="0 0 0" xyz="0 0 0" />
+        <material name="${prefix}black" />
+      </visual>
       <inertial>
         <mass value="0.194" />
-        <origin xyz="0.005 -0.001 0.016" />
-        <inertia
-          ixx="0.000189" ixy="0.000005" ixz="0.000054"
-          iyx="0.000005" iyy="0.000213" iyz="0.000003"
-          izx="0.000054" izy="0.000003" izz="0.000067" />
+        <origin xyz="0 0 0.0165" />
+        <inertia
+          ixx="0.000037"
+          ixy="0"
+          ixz="0"
+          iyy="0.000037"
+          iyz="0"
+          izz="0.0000388"
+        />
       </inertial>
     </link>
@@ -57,34 +69,20 @@
       <visual>
         <geometry>
-          <mesh filename="package://alpha_description/meshes/M2.stl" />
-        </geometry>
-        <origin rpy="0 0 0" xyz="0 0 0" />
-        <material name="${prefix}black" />
-      </visual>
-      <collision>
-        <geometry>
-          <cylinder length="0.145" radius="0.020" />
-        </geometry>
-        <origin rpy="0 0 0" xyz="-0.02 0 -0.0725" />
-      </collision>
-      <collision>
-        <geometry>
-          <cylinder length="0.040" radius="0.020" />
-        </geometry>
-        <origin rpy="1.5707 0 0" xyz="0 0 0" />
-      </collision>
-      <collision>
-        <geometry>
-          <cylinder length="0.040" radius="0.020" />
-        </geometry>
-        <origin rpy="1.5707 0 0" xyz="-0.040 0 -0.1453" />
-      </collision>
+          <mesh filename="file://$(find alpha_description)/meshes/M2.stl" />
+        </geometry>
+        <origin rpy="0 0 0" xyz="0 0 0" />
+        <material name="${prefix}black" />
+      </visual>
       <inertial>
         <mass value="0.429" />
-        <origin xyz="0.073 0.0 0.0" />
-        <inertia
-          ixx="0.000087" ixy="-0.000076" ixz="-0.00001"
-          iyx="-0.000076" iyy="0.00319" iyz="0"
-          izx="-0.00001" izy="0" izz="0.003212" />
+        <origin xyz="-0.02 0 -0.0725" />
+        <inertia
+          ixx="0.0008907"
+          ixy="0"
+          ixz="0"
+          iyy="0.0008907"
+          iyz="0"
+          izz="0.0000858"
+        />
       </inertial>
     </link>
@@ -92,22 +90,20 @@
       <visual>
         <geometry>
-          <mesh filename="package://alpha_description/meshes/M2-1-3.stl" />
-        </geometry>
-        <origin rpy="0 0 0" xyz="0 0 0" />
-        <material name="${prefix}black" />
-      </visual>
-      <collision>
-        <geometry>
-          <cylinder length="0.033" radius="0.020" />
-        </geometry>
-        <origin rpy="0 0 0" xyz="0.02 0 0.0165" />
-      </collision>
+          <mesh filename="file://$(find alpha_description)/meshes/M2-1-3.stl" />
+        </geometry>
+        <origin rpy="0 0 0" xyz="0 0 0" />
+        <material name="${prefix}black" />
+      </visual>
       <inertial>
         <mass value="0.115" />
-        <origin xyz="0.017 -0.026 -0.002" />
-        <inertia
-          ixx="0.00012" ixy="-0.000061" ixz="-0.000001"
-          iyx="-0.000061" iyy="0.000062" iyz="0"
-          izx="-0.000001" izy="0" izz="0.000156" />
+        <origin xyz="0.02 0 0.0165" />
+        <inertia
+          ixx="0.0000219"
+          ixy="0"
+          ixz="0"
+          iyy="0.0000219"
+          iyz="0"
+          izz="0.000023"
+        />
       </inertial>
     </link>
@@ -116,36 +112,58 @@
         <geometry>
           <mesh
-            filename="package://alpha_description/meshes/RS1-100-101-123.stl" />
+            filename="file://$(find alpha_description)/meshes/RS1-100-101-123.stl" />
         </geometry>
         <origin rpy="0 -1.5707 0" xyz="0 0 0" />
         <material name="${prefix}black" />
       </visual>
-      <collision>
-        <geometry>
-          <cylinder length="0.10975" radius="0.020" />
-        </geometry>
-        <origin rpy="0 0 0" xyz="0.00 0 0.054875" />
-      </collision>
       <inertial>
         <mass value="0.333" />
-        <origin xyz="0.0 0.003 -0.098" />
-        <inertia
-          ixx="0.003709" ixy="0.000002" ixz="-0.000004"
-          iyx="0.000002" iyy="0.003734" iyz="0"
-          izx="-0.000004" izy="0" izz="0.000079" />
+        <origin xyz="0 0 0.054875" />
+        <inertia
+          ixx="0.0003676"
+          ixy="0"
+          ixz="0"
+          iyy="0.0003676"
+          iyz="0"
+          izz="0.0000666"
+        />
       </inertial>
     </link>
     <link name="${prefix}ee_base_link">
-      <inertial>
-        <mass value="2e-06" />
-        <inertia ixx="1.1e-09" ixy="0" ixz="0" iyy="1.1e-09" iyz="0"
-          izz="1.1e-09" />
+      <visual>
+        <origin rpy="0 0 0" xyz="0 0 0" />
+        <geometry>
+          <box size="0.001 0.001 0.001" />
+        </geometry>
+      </visual>
+      <inertial>
+        <mass value="0.0001" />
+        <inertia
+          ixx="0.0001"
+          ixy="0"
+          ixz="0"
+          iyy="0.0001"
+          iyz="0"
+          izz="0.0001"
+        />
       </inertial>
     </link>
     <link name="${prefix}push_rod">
-      <inertial>
-        <mass value="2e-06" />
-        <inertia ixx="1.1e-09" ixy="0" ixz="0" iyy="1.1e-09" iyz="0"
-          izz="1.1e-09" />
+      <visual>
+        <origin rpy="0 0 0" xyz="0 0 0" />
+        <geometry>
+          <box size="0.001 0.001 0.001" />
+        </geometry>
+      </visual>
+      <inertial>
+        <mass value="0.0001" />
+        <inertia
+          ixx="0.0001"
+          ixy="0"
+          ixz="0"
+          iyy="0.0001"
+          iyz="0"
+          izz="0.0001"
+        />
       </inertial>
     </link>
@@ -205,5 +223,5 @@
     </joint>
     <xacro:include
-      filename="$(find alpha_description)/urdf/end_effectors/standard_jaws.urdf.xacro" />
+      filename="$(find angler_description)/urdf/end_effectors/standard_jaws.urdf.xacro" />
     <xacro:alpha_standard_jaws parent="${prefix}ee_base_link"
       prefix="${prefix}standard_jaws_"

File: angler_description/urdf/bluerov2_heavy_modified.urdf.xacro (robot description, xacro)
@@ -19,5 +19,5 @@
         <geometry>
           <mesh
-            filename="package://angler_description/meshes/bluerov2/bluerov2_heavy_modified.dae"
+            filename="package://angler_description/meshes/bluerov2_heavy_modified.dae"
             scale="0.025 0.025 0.025"
           />
@@ -46,5 +46,5 @@
       <visual>
         <geometry>
-          <mesh filename="package://angler_description/meshes/bluerov2/t200_ccw_prop.dae" />
+          <mesh filename="package://angler_description/meshes/t200_ccw_prop.dae" />
         </geometry>
         <origin rpy="-1.571 0 0" xyz="0 0 0" />
@@ -65,5 +65,5 @@
       <visual>
         <geometry>
-          <mesh filename="package://angler_description/meshes/bluerov2/t200_ccw_prop.dae" />
+          <mesh filename="package://angler_description/meshes/t200_ccw_prop.dae" />
         </geometry>
         <origin rpy="-1.571 0 0" xyz="0 0 0" />
@@ -84,5 +84,5 @@
       <visual>
         <geometry>
-          <mesh filename="package://angler_description/meshes/bluerov2/t200_cw_prop.dae" />
+          <mesh filename="package://angler_description/meshes/t200_cw_prop.dae" />
         </geometry>
         <origin rpy="1.571 0 0" xyz="0 0 0" />
@@ -103,5 +103,5 @@
       <visual>
         <geometry>
-          <mesh filename="package://angler_description/meshes/bluerov2/t200_cw_prop.dae" />
+          <mesh filename="package://angler_description/meshes/t200_cw_prop.dae" />
         </geometry>
         <origin rpy="1.571 0 0" xyz="0 0 0" />
@@ -122,5 +122,5 @@
       <visual>
         <geometry>
-          <mesh filename="package://angler_description/meshes/bluerov2/t200_ccw_prop.dae" />
+          <mesh filename="package://angler_description/meshes/t200_ccw_prop.dae" />
         </geometry>
         <origin rpy="-1.571 0 1.571" xyz="0 0 0" />
@@ -141,5 +141,5 @@
       <visual>
         <geometry>
-          <mesh filename="package://angler_description/meshes/bluerov2/t200_cw_prop.dae" />
+          <mesh filename="package://angler_description/meshes/t200_cw_prop.dae" />
         </geometry>
         <origin rpy="1.571 0 1.571" xyz="0 0 0" />
@@ -160,5 +160,5 @@
       <visual>
         <geometry>
-          <mesh filename="package://angler_description/meshes/bluerov2/t200_cw_prop.dae" />
+          <mesh filename="package://angler_description/meshes/t200_cw_prop.dae" />
         </geometry>
         <origin rpy="1.571 0 1.571" xyz="0 0 0" />
@@ -179,5 +179,5 @@
       <visual>
         <geometry>
-          <mesh filename="package://angler_description/meshes/bluerov2/t200_ccw_prop.dae" />
+          <mesh filename="package://angler_description/meshes/t200_ccw_prop.dae" />
         </geometry>
         <origin rpy="-1.571 0 1.571" xyz="0 0 0" />
@@ -185,8 +185,20 @@
     </link>
     <link name="${prefix}manipulator_mount_link">
-      <inertial>
-        <mass value="2e-06" />
-        <inertia ixx="1.1e-09" ixy="0" ixz="0" iyy="1.1e-09" iyz="0"
-          izz="1.1e-09" />
+      <visual>
+        <origin rpy="0 0 0" xyz="0 0 0" />
+        <geometry>
+          <box size="0.001 0.001 0.001" />
+        </geometry>
+      </visual>
+      <inertial>
+        <mass value="0.0001" />
+        <inertia
+          ixx="0.0001"
+          ixy="0"
+          ixz="0"
+          iyy="0.0001"
+          iyz="0"
+          izz="0.0001"
+        />
       </inertial>
     </link>

File: angler_description/urdf/end_effectors/standard_jaws.urdf.xacro (robot description, xacro)
@@ -10,12 +10,18 @@
         <geometry>
           <mesh
-            filename="package://alpha_description/meshes/end_effectors/RS1-124.stl" />
+            filename="file://$(find alpha_description)/meshes/end_effectors/RS1-124.stl" />
         </geometry>
         <material name="${prefix}black" />
       </visual>
       <inertial>
-        <mass value="2e-06" />
-        <inertia ixx="1.1e-09" ixy="0" ixz="0" iyy="1.1e-09" iyz="0"
-          izz="1.1e-09" />
+        <mass value="0.0001" />
+        <inertia
+          ixx="0.0001"
+          ixy="0"
+          ixz="0"
+          iyy="0.0001"
+          iyz="0"
+          izz="0.0001"
+        />
       </inertial>
     </link>
@@ -24,19 +30,19 @@
         <geometry>
           <mesh
-            filename="package://alpha_description/meshes/end_effectors/RS1-130.stl" />
+            filename="file://$(find alpha_description)/meshes/end_effectors/RS1-130.stl" />
         </geometry>
         <material name="${prefix}black" />
         <origin xyz="0 0 0" rpy="0 0 0" />
       </visual>
-      <collision>
-        <geometry>
-          <box size="0.012 0.03 0.09" />
-        </geometry>
-        <origin xyz="0.0 -0.008 0.045" rpy="0 0 0" />
-      </collision>
       <inertial>
-        <mass value="2e-06" />
-        <inertia ixx="1.1e-09" ixy="0" ixz="0" iyy="1.1e-09" iyz="0"
-          izz="1.1e-09" />
+        <mass value="0.0001" />
+        <inertia
+          ixx="0.0001"
+          ixy="0"
+          ixz="0"
+          iyy="0.0001"
+          iyz="0"
+          izz="0.0001"
+        />
       </inertial>
     </link>
@@ -45,19 +51,19 @@
         <geometry>
           <mesh
-            filename="package://alpha_description/meshes/end_effectors/RS1-139.stl" />
+            filename="file://$(find alpha_description)/meshes/end_effectors/RS1-139.stl" />
         </geometry>
         <material name="${prefix}black" />
         <origin xyz="0 0 0" rpy="0 0 0" />
       </visual>
-      <collision>
-        <geometry>
-          <box size="0.012 0.03 0.09" />
-        </geometry>
-        <origin xyz="0.0 0.008 0.045" rpy="0 0 0" />
-      </collision>
       <inertial>
-        <mass value="2e-06" />
-        <inertia ixx="1.1e-09" ixy="0" ixz="0" iyy="1.1e-09" iyz="0"
-          izz="1.1e-09" />
+        <mass value="0.0001" />
+        <inertia
+          ixx="0.0001"
+          ixy="0"
+          ixz="0"
+          iyy="0.0001"
+          iyz="0"
+          izz="0.0001"
+        />
       </inertial>
     </link>
