Commit message: More bug fixes from cleanup

File: angler_description/xacro/bluerov2_heavy_alpha/config.xacro (robot description, xacro)
@@ -27,5 +27,5 @@
     serial_port="$(arg serial_port)"
     state_update_frequency="$(arg state_update_frequency)"
-    initial_positions_file="$(arg initial_positions_file)"
+    initial_positions_file="/bluerov2_heavy_alpha/$(arg initial_positions_file)"
     description_package="${description_package}"
     use_sim="${use_sim}"
@@ -39,5 +39,5 @@
       description_package="${description_package}"
       namespace="$(arg namespace)"
-      controllers_file="$(arg controllers_file)" />
+      controllers_file="bluerov2_heavy_alpha/$(arg controllers_file)" />
   </xacro:if>
 </robot>

File: angler_description/xacro/bluerov2_heavy_alpha/urdf.xacro (robot description, xacro)
@@ -21,8 +21,54 @@
       </inertial>
     </link>
+    <link name="${prefix}ballast_link">
+      <inertial>
+        <mass value="0.0001" />
+        <inertia
+          ixx="0.0001"
+          ixy="0"
+          ixz="0"
+          iyy="0.0001"
+          iyz="0"
+          izz="0.0001"
+        />
+      </inertial>
+      <!-- Front-Left -->
+      <collision>
+        <geometry>
+          <box size="0.15 0.15 0.035" />
+        </geometry>
+        <origin rpy="0 0 0" xyz="0.118 0.21 0.05" />
+      </collision>
+      <!-- Front-Right -->
+      <collision>
+        <geometry>
+          <box size="0.15 0.15 0.08" />
+        </geometry>
+        <origin rpy="0 0 0" xyz="0.118 -0.21 0.05" />
+      </collision>
+      <!-- Left -->
+      <collision>
+        <geometry>
+          <box size="0.1 0.1 0.0225" />
+        </geometry>
+        <origin rpy="0 0 0" xyz="0 0.10375 0.05" />
+      </collision>
+      <!-- Right -->
+      <collision>
+        <geometry>
+          <box size="0.1 0.1 0.0225" />
+        </geometry>
+        <origin rpy="0 0 0" xyz="0 -0.10375 0.05" />
+      </collision>
+    </link>
     <joint name="${prefix}manipulator_mount_joint" type="fixed">
       <origin rpy="0 0 0" xyz="0.24 -0.099 0.029" />
       <parent link="${prefix}base_link" />
       <child link="${prefix}manipulator_mount_link" />
+    </joint>
+    <joint name="${prefix}ballast_joint" type="fixed">
+      <origin rpy="0 0 0" xyz="0 0 0" />
+      <parent link="${prefix}base_link" />
+      <child link="${prefix}ballast_link" />
     </joint>
     <!-- Imports -->
